File: logic.kicad_sch (KiCad schematic)
At the start: 68 parts, among them J5 HanRun_HR911105A, Q24 2N7002, Q25 AO3401A, U10 LAN8720A, U11 74HC595, U17 N066-6448TSWEG03-H28, U8 SY8120B1ABC, U9 ESP32-WROOM-32E

Commit message: Partial layout
Parts:
- gave numbers to parts that had none: 2
Connections:
- net +3.3V is gone; now on net +3V3: C66.1, J5.4 (TCT), J5.5 (RCT), R66.1, R68.1, R70.1, R71.1
Changed lines of the file:
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@@
-    (pin "1")
-  )
-  (symbol (lib_id "power:+3.3V") (at 100.33 121.92 0) (unit 1)
-    (in_bom yes) (on_board yes) (fields_autoplaced)
-    (property "Reference" "#PWR0217" (id 0) (at 100.33 125.73 0)
-      (effects (font (size 1.27 1.27)) hide)
-    )
-    (property "Value" "+3.3V" (id 1) (at 100.33 118.3442 0))
-    (property "Footprint" "" (id 2) (at 100.33 121.92 0)
-      (effects (font (size 1.27 1.27)) hide)
-    )
-    (property "Datasheet" "" (id 3) (at 100.33 121.92 0)
-      (effects (font (size 1.27 1.27)) hide)
-    )
     (pin "1")
   )
@@
     (pin "9")
   )
+  (symbol (lib_id "power:+3V3") (at 100.33 121.92 0) (unit 1)
+    (in_bom yes) (on_board yes) (fields_autoplaced)
+    (property "Reference" "#PWR0217" (id 0) (at 100.33 125.73 0)
+      (effects (font (size 1.27 1.27)) hide)
+    )
+    (property "Value" "+3V3" (id 1) (at 100.33 118.3442 0))
+    (property "Footprint" "" (id 2) (at 100.33 121.92 0)
+      (effects (font (size 1.27 1.27)) hide)
+    )
+    (property "Datasheet" "" (id 3) (at 100.33 121.92 0)
+      (effects (font (size 1.27 1.27)) hide)
+    )
+    (pin "1")
+  )
   (symbol (lib_id "Device:R_Small") (at 110.49 151.13 270) (unit 1)
     (in_bom yes) (on_board yes)
@@
   (symbol (lib_id "power:GND") (at 266.7 86.36 0) (unit 1)
     (in_bom yes) (on_board yes) (fields_autoplaced)
-    (property "Reference" "#PWR?" (id 0) (at 266.7 92.71 0)
+    (property "Reference" "#PWR0299" (id 0) (at 266.7 92.71 0)
       (effects (font (size 1.27 1.27)) hide)
     )
@@
   (symbol (lib_id "power:+3V3") (at 271.78 71.12 0) (unit 1)
     (in_bom yes) (on_board yes) (fields_autoplaced)
-    (property "Reference" "#PWR?" (id 0) (at 271.78 74.93 0)
+    (property "Reference" "#PWR0297" (id 0) (at 271.78 74.93 0)
       (effects (font (size 1.27 1.27)) hide)
     )
@@
   (symbol (lib_id "Device:R_Small") (at 271.78 74.93 0) (unit 1)
     (in_bom yes) (on_board yes) (fields_autoplaced)
-    (property "Reference" "R?" (id 0) (at 273.2786 74.0953 0)
+    (property "Reference" "R118" (id 0) (at 273.2786 74.0953 0)
       (effects (font (size 1.27 1.27)) (justify left))
     )
@@
   (symbol (lib_id "power:GND") (at 271.78 91.44 0) (unit 1)
     (in_bom yes) (on_board yes) (fields_autoplaced)
-    (property "Reference" "#PWR?" (id 0) (at 271.78 97.79 0)
+    (property "Reference" "#PWR0298" (id 0) (at 271.78 97.79 0)
       (effects (font (size 1.27 1.27)) hide)
     )
@@
   (symbol (lib_id "Switch_MountingPin:SW_Push_MountingPin") (at 271.78 85.09 270) (unit 1)
     (in_bom yes) (on_board yes) (fields_autoplaced)
-    (property "Reference" "SW?" (id 0) (at 275.463 84.2553 90)
-      (effects (font (size 1.27 1.27)) (justify left))
-    )
+    (property "Reference" "SW2" (id 0) (at 275.463 84.2553 90)
+      (effects (font (size 1.27 1.27)) (justify left))
+    )
