File: dc-usv.kicad_sch (KiCad schematic)
At the start: 3 parts

Commit message: Add 3d models
Parts:
- added PANEL?: Backpanel, Panels:Backpanel, symbol Case:Panel
- added PANEL?: Frontpanel, Panels:Frontpanel, symbol Case:Panel
Changed lines of the file:
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@@
+    )
+  )
+  (symbol (lib_id "Case:Panel") (at 48.26 33.02 0) (unit 1)
+    (in_bom yes) (on_board yes)
+    (property "Reference" "PANEL?" (id 0) (at 44.45 30.48 0)
+      (effects (font (size 1.27 1.27)) (justify left))
+    )
+    (property "Value" "Backpanel" (id 1) (at 43.18 33.02 0)
+      (effects (font (size 1.27 1.27)) (justify left))
+    )
+    (property "Footprint" "Panels:Backpanel" (id 2) (at 48.26 33.02 0)
+      (effects (font (size 1.27 1.27)) hide)
+    )
+    (property "Datasheet" "" (id 3) (at 48.26 33.02 0)
+      (effects (font (size 1.27 1.27)) hide)
+    )
+  )
+  (symbol (lib_id "Case:Panel") (at 35.56 33.02 0) (unit 1)
+    (in_bom yes) (on_board yes)
+    (property "Reference" "PANEL?" (id 0) (at 31.75 30.48 0)
+      (effects (font (size 1.27 1.27)) (justify left))
+    )
+    (property "Value" "Frontpanel" (id 1) (at 30.48 33.02 0)
+      (effects (font (size 1.27 1.27)) (justify left))
+    )
+    (property "Footprint" "Panels:Frontpanel" (id 2) (at 35.56 33.02 0)
+      (effects (font (size 1.27 1.27)) hide)
+    )
+    (property "Datasheet" "" (id 3) (at 35.56 33.02 0)
+      (effects (font (size 1.27 1.27)) hide)
     )
   )
@@
       (reference "L4") (unit 1) (value "4.7uH") (footprint "Inductor_SMD:L_Bourns_SRP7028A_7.3x6.6mm")
     )
+    (path "/c4b014eb-17fb-4187-8a93-f75b025805d7"
+      (reference "PANEL?") (unit 1) (value "Backpanel") (footprint "Panels:Backpanel")
+    )
+    (path "/f60fd6cd-f5a9-4404-bb7e-7667eeafd907"
+      (reference "PANEL?") (unit 1) (value "Frontpanel") (footprint "Panels:Frontpanel")
+    )
     (path "/aa145c2f-e167-4de3-92bf-3e0d0ae2fb67/8dec12cb-4e13-410a-a8ed-ba1ad46e962f"

Commit message: Fix reversed debug USB TVS
Parts:
- gave numbers to parts that had none: 2
Changed lines of the file:
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@@
   (symbol (lib_id "Case:Panel") (at 48.26 33.02 0) (unit 1)
     (in_bom yes) (on_board yes)
-    (property "Reference" "PANEL?" (id 0) (at 44.45 30.48 0)
+    (property "Reference" "PANEL2" (id 0) (at 44.45 30.48 0)
       (effects (font (size 1.27 1.27)) (justify left))
     )
@@
   (symbol (lib_id "Case:Panel") (at 35.56 33.02 0) (unit 1)
     (in_bom yes) (on_board yes)
-    (property "Reference" "PANEL?" (id 0) (at 31.75 30.48 0)
+    (property "Reference" "PANEL1" (id 0) (at 31.75 30.48 0)
       (effects (font (size 1.27 1.27)) (justify left))
     )
@@
       (reference "L4") (unit 1) (value "4.7uH") (footprint "Inductor_SMD:L_Bourns_SRP7028A_7.3x6.6mm")
     )
+    (path "/f60fd6cd-f5a9-4404-bb7e-7667eeafd907"
+      (reference "PANEL1") (unit 1) (value "Frontpanel") (footprint "Panels:Frontpanel")
+    )
     (path "/c4b014eb-17fb-4187-8a93-f75b025805d7"
-      (reference "PANEL?") (unit 1) (value "Backpanel") (footprint "Panels:Backpanel")
-    )
-    (path "/f60fd6cd-f5a9-4404-bb7e-7667eeafd907"
-      (reference "PANEL?") (unit 1) (value "Frontpanel") (footprint "Panels:Frontpanel")
+      (reference "PANEL2") (unit 1) (value "Backpanel") (footprint "Panels:Backpanel")
     )
     (path "/aa145c2f-e167-4de3-92bf-3e0d0ae2fb67/8dec12cb-4e13-410a-a8ed-ba1ad46e962f"
